Commit message: Enabled 2F-140 gripper be simulated on Gazebo Classic, but suspecting collision issue, has implemented work around to disable collision of the affected link in Gazebo.
Signed-off-by: laidvi <laidvi@schaeffler.com>

File: robotiq_description/urdf/2f_140.ros2_control.xacro (robot description, xacro)
@@ -5,4 +5,5 @@
         prefix
         sim_ignition:=false
+        sim_gazebo:=false
         sim_isaac:=false
         isaac_joint_commands:=/isaac_joint_commands
@@ -22,4 +23,7 @@
                     <plugin>ign_ros2_control/IgnitionSystem</plugin>
                 </xacro:if>
+                <xacro:if value="${sim_gazebo}">
+                    <plugin>gazebo_ros2_control/GazeboSystem</plugin>
+                </xacro:if>
                 <xacro:if value="${use_fake_hardware}">
                     <plugin>mock_components/GenericSystem</plugin>
@@ -38,4 +42,5 @@
             <!-- With Ignition or Hardware, they handle mimic joints, so we only need this command interface activated -->
             <joint name="${prefix}finger_joint">
+                <!-- <command_interface name="effort" /> -->
                 <command_interface name="position" />
                 <state_interface name="position">
@@ -43,11 +48,12 @@
                 </state_interface>
                 <state_interface name="velocity"/>
+                <!-- <state_interface name="effort" /> -->
             </joint>
             <!-- When simulating we need to include the rest of the gripper joints -->
-            <xacro:if value="${use_fake_hardware or sim_isaac or sim_ignition}">
+            <xacro:if value="${use_fake_hardware or sim_isaac or sim_ignition or sim_gazebo}">
                 <joint name="${prefix}left_inner_knuckle_joint">
                     <param name="mimic">${prefix}finger_joint</param>
                     <param name="multiplier">-1</param>
-                    <xacro:unless value="${sim_ignition}">
+                    <xacro:unless value="${sim_ignition and sim_gazebo}">
                         <command_interface name="position"/>
                         <state_interface name="position"/>
@@ -58,5 +64,5 @@
                     <param name="mimic">${prefix}finger_joint</param>
                     <param name="multiplier">1</param>
-                    <xacro:unless value="${sim_ignition}">
+                    <xacro:unless value="${sim_ignition and sim_gazebo}">
                         <command_interface name="position"/>
                         <state_interface name="position"/>
@@ -67,5 +73,5 @@
                     <param name="mimic">${prefix}finger_joint</param>
                     <param name="multiplier">-1</param>
-                    <xacro:unless value="${sim_ignition}">
+                    <xacro:unless value="${sim_ignition and sim_gazebo}">
                         <command_interface name="position"/>
                         <state_interface name="position"/>
@@ -76,5 +82,5 @@
                     <param name="mimic">${prefix}finger_joint</param>
                     <param name="multiplier">-1</param>
-                    <xacro:unless value="${sim_ignition}">
+                    <xacro:unless value="${sim_ignition and sim_gazebo}">
                         <command_interface name="position"/>
                         <state_interface name="position"/>
@@ -85,5 +91,5 @@
                     <param name="mimic">${prefix}finger_joint</param>
                     <param name="multiplier">1</param>
-                    <xacro:unless value="${sim_ignition}">
+                    <xacro:unless value="${sim_ignition and sim_gazebo}">
                         <command_interface name="position"/>
                         <state_interface name="position"/>
@@ -93,5 +99,5 @@
             </xacro:if>
             <!-- Only add this with fake hardware mode -->
-            <xacro:unless value="${sim_ignition or sim_isaac}">
+            <xacro:unless value="${sim_ignition or sim_isaac or sim_gazebo}">
                 <gpio name="reactivate_gripper">
                     <command_interface name="reactivate_gripper_cmd" />

File: robotiq_description/urdf/robotiq_2f_140_gripper.urdf.xacro (robot description, xacro)
@@ -2,10 +2,70 @@
 <robot xmlns:xacro="http://wiki.ros.org/xacro" name="robotiq_gripper">
     <!-- parameters -->
+    <xacro:arg name="sim_gazebo" default="false" />
     <xacro:arg name="use_fake_hardware" default="true" />
+    <xacro:arg name="prefix" default="" />
+    <xacro:arg name="simulation_controllers" default="" />
+    <xacro:arg name="generate_ros2_control_tag" default="true" />
     <!-- Import macros -->
     <xacro:include filename="$(find robotiq_description)/urdf/robotiq_2f_140_macro.urdf.xacro" />
     <link name="world" />
-    <xacro:robotiq_gripper name="RobotiqGripperHardwareInterface" prefix="" parent="world" use_fake_hardware="$(arg use_fake_hardware)">
+    <xacro:robotiq_gripper
+        name="RobotiqGripperHardwareInterface"
+        prefix="$(arg prefix)"
+        parent="world"
+        sim_gazebo="$(arg sim_gazebo)"
+        use_fake_hardware="$(arg use_fake_hardware)"
+        include_ros2_control="$(arg generate_ros2_control_tag)">
         <origin xyz="0 0 0" rpy="0 0 0" />
     </xacro:robotiq_gripper>
+    <xacro:if value="$(arg sim_gazebo)">
+        <gazebo>
+            <plugin filename="libgazebo_ros2_control.so" name="gazebo_ros2_control">
+                <robot_param_node>robot_state_publisher</robot_param_node>
+                <parameters>$(arg simulation_controllers)</parameters>
+            </plugin>
+            <plugin filename="libroboticsgroup_upatras_gazebo_mimic_joint_plugin.so"
+                name="$(arg prefix)left_inner_knuckle_joint_mmmmmmmmmmmmmmmm">
+                <joint>$(arg prefix)finger_joint</joint>
+                <mimicJoint>$(arg prefix)left_inner_knuckle_joint</mimicJoint>
+                <multiplier>-1.0</multiplier>
+            </plugin>
+            <plugin filename="libroboticsgroup_upatras_gazebo_mimic_joint_plugin.so"
+                name="$(arg prefix)left_inner_finger_joint">
+                <joint>$(arg prefix)finger_joint</joint>
+                <mimicJoint>$(arg prefix)left_inner_finger_joint</mimicJoint>
+                <multiplier>1.0</multiplier>
+            </plugin>
+            <plugin filename="libroboticsgroup_upatras_gazebo_mimic_joint_plugin.so"
+                name="$(arg prefix)right_outer_knuckle_joint">
+                <joint>$(arg prefix)finger_joint</joint>
+                <mimicJoint>$(arg prefix)right_outer_knuckle_joint</mimicJoint>
+                <multiplier>-1.0</multiplier>
+            </plugin>
+            <plugin filename="libroboticsgroup_upatras_gazebo_mimic_joint_plugin.so"
+                name="$(arg prefix)right_inner_knuckle_joint">
+                <joint>$(arg prefix)finger_joint</joint>
+                <mimicJoint>$(arg prefix)right_inner_knuckle_joint</mimicJoint>
+                <multiplier>-1.0</multiplier>
+            </plugin>
+            <plugin filename="libroboticsgroup_upatras_gazebo_mimic_joint_plugin.so"
+                name="$(arg prefix)right_inner_finger_joint">
+                <joint>$(arg prefix)finger_joint</joint>
+                <mimicJoint>$(arg prefix)right_inner_finger_joint</mimicJoint>
+                <multiplier>1.0</multiplier>
+            </plugin>
+        </gazebo>
+        <gazebo reference="left_inner_knuckle">
+            <selfCollide>false</selfCollide>
+        </gazebo>
+        <gazebo reference="left_outer_knuckle">
+            <selfCollide>false</selfCollide>
+        </gazebo>
+        <gazebo reference="left_inner_finger">
+            <selfCollide>false</selfCollide>
+        </gazebo>
+        <gazebo reference="left_outer_finger">
+            <selfCollide>true</selfCollide>
+        </gazebo>
+    </xacro:if>
 </robot>

File: robotiq_description/urdf/robotiq_2f_140_macro.urdf.xacro (robot description, xacro)
@@ -7,4 +7,5 @@
         *origin
         sim_ignition:=false
+        sim_gazebo:=false
         sim_isaac:=false
         isaac_joint_commands:=/isaac_joint_commands
@@ -21,4 +22,5 @@
                 name="${name}" prefix="${prefix}"
                 sim_ignition="${sim_ignition}"
+                sim_gazebo="${sim_gazebo}"
                 sim_isaac="${sim_isaac}"
                 isaac_joint_commands="${isaac_joint_commands}"
