Commit message: Disable base link collision
Signed-off-by: laidvi <laidvi@schaeffler.com>

File: robotiq_description/urdf/robotiq_2f_140_gripper.urdf.xacro (robot description, xacro)
@@ -26,5 +26,5 @@
             </plugin>
             <plugin filename="libroboticsgroup_upatras_gazebo_mimic_joint_plugin.so"
-                name="$(arg prefix)left_inner_knuckle_joint_mmmmmmmmmmmmmmmm">
+                name="$(arg prefix)left_inner_knuckle_joint">
                 <joint>$(arg prefix)finger_joint</joint>
                 <mimicJoint>$(arg prefix)left_inner_knuckle_joint</mimicJoint>

File: robotiq_description/urdf/robotiq_2f_140_macro.urdf.xacro (robot description, xacro)
@@ -54,6 +54,8 @@
         <collision>
           <origin xyz="0 0 0" rpy="0 0 0" />
+          <!-- NOTE: This collision stl will cause collision in Gazebo -->
           <geometry>
-            <mesh filename="file://$(find robotiq_description)/meshes/collision/2f_140/robotiq_2f_140_base_link.stl" />
+            <cylinder length="0.006" radius="0.2"/>
+            <!-- <mesh filename="file://$(find robotiq_description)/meshes/collision/2f_140/robotiq_2f_140_base_link.stl" /> -->
           </geometry>
         </collision>
