Commit message: Added damping at each revolute joint to fix the damping effect.
Signed-off-by: laidvi <laidvi@schaeffler.com>

File: robotiq_description/urdf/robotiq_2f_140.xacro (robot description, xacro)
@@ -7,15 +7,16 @@
         <mass value="0.00853198276973456" />
         <inertia
-            ixx="2.89328108496468E-06"
-            ixy="-1.57935047237397E-19"
-            ixz="-1.93980378593255E-19"
-            iyy="1.86719750325683E-06"
-            iyz="-1.21858577871576E-06"
-            izz="1.21905238907251E-06" />
-      </inertial>
-      <visual>
-        <origin xyz="0 0 0" rpy="0 0 0" />
-        <geometry>
-          <mesh filename="file://$(find robotiq_description)/meshes/visual/2f_140/robotiq_2f_${stroke}_outer_knuckle.stl" />
+          ixx="2.89328108496468E-06"
+          ixy="-1.57935047237397E-19"
+          ixz="-1.93980378593255E-19"
+          iyy="1.86719750325683E-06"
+          iyz="-1.21858577871576E-06"
+          izz="1.21905238907251E-06" />
+      </inertial>
+      <visual>
+        <origin xyz="0 0 0" rpy="0 0 0" />
+        <geometry>
+          <mesh
+            filename="file://$(find robotiq_description)/meshes/visual/2f_140/robotiq_2f_${stroke}_outer_knuckle.stl" />
         </geometry>
         <material name="">
@@ -26,5 +27,6 @@
         <origin xyz="0 0 0" rpy="0 0 0" />
         <geometry>
-          <mesh filename="file://$(find robotiq_description)/meshes/collision/2f_140/robotiq_2f_${stroke}_outer_knuckle.stl" />
+          <mesh
+            filename="file://$(find robotiq_description)/meshes/collision/2f_140/robotiq_2f_${stroke}_outer_knuckle.stl" />
         </geometry>
       </collision>
@@ -37,15 +39,16 @@
         <mass value="0.022614240507152" />
         <inertia
-            ixx="1.52518312458174E-05"
-            ixy="9.76583423954399E-10"
-            ixz="-5.43838577022588E-10"
-            iyy="6.17694243867776E-06"
-            iyz="6.78636130740228E-06"
-            izz="1.16494917907219E-05" />
-      </inertial>
-      <visual>
-        <origin xyz="0 0 0" rpy="0 0 0" />
-        <geometry>
-          <mesh filename="file://$(find robotiq_description)/meshes/visual/2f_140/robotiq_2f_${stroke}_outer_finger.stl" />
+          ixx="1.52518312458174E-05"
+          ixy="9.76583423954399E-10"
+          ixz="-5.43838577022588E-10"
+          iyy="6.17694243867776E-06"
+          iyz="6.78636130740228E-06"
+          izz="1.16494917907219E-05" />
+      </inertial>
+      <visual>
+        <origin xyz="0 0 0" rpy="0 0 0" />
+        <geometry>
+          <mesh
+            filename="file://$(find robotiq_description)/meshes/visual/2f_140/robotiq_2f_${stroke}_outer_finger.stl" />
         </geometry>
         <material name="">
@@ -56,5 +59,6 @@
         <origin xyz="0 0 0" rpy="0 0 0" />
         <geometry>
-          <mesh filename="file://$(find robotiq_description)/meshes/collision/2f_140/robotiq_2f_${stroke}_outer_finger.stl" />
+          <mesh
+            filename="file://$(find robotiq_description)/meshes/collision/2f_140/robotiq_2f_${stroke}_outer_finger.stl" />
         </geometry>
       </collision>
@@ -67,15 +71,16 @@
         <mass value="0.0271177346495152" />
         <inertia
-            ixx="2.61910379223783E-05"
-            ixy="-2.43616858946494E-07"
-            ixz="-6.37789906117123E-09"
-            iyy="2.8270243746167E-06"
-            iyz="-5.37200748039765E-07"
-            izz="2.83695868220296E-05" />
-      </inertial>
-      <visual>
-        <origin xyz="0 0 0" rpy="0 0 0" />
-        <geometry>
-          <mesh filename="file://$(find robotiq_description)/meshes/visual/2f_140/robotiq_2f_${stroke}_inner_knuckle.stl" />
+          ixx="2.61910379223783E-05"
+          ixy="-2.43616858946494E-07"
+          ixz="-6.37789906117123E-09"
+          iyy="2.8270243746167E-06"
+          iyz="-5.37200748039765E-07"
+          izz="2.83695868220296E-05" />
+      </inertial>
+      <visual>
+        <origin xyz="0 0 0" rpy="0 0 0" />
+        <geometry>
+          <mesh
+            filename="file://$(find robotiq_description)/meshes/visual/2f_140/robotiq_2f_${stroke}_inner_knuckle.stl" />
         </geometry>
         <material name="">
@@ -86,5 +91,6 @@
         <origin xyz="0 0 0" rpy="0 0 0" />
         <geometry>
-          <mesh filename="file://$(find robotiq_description)/meshes/collision/2f_140/robotiq_2f_${stroke}_inner_knuckle.stl" />
+          <mesh
+            filename="file://$(find robotiq_description)/meshes/collision/2f_140/robotiq_2f_${stroke}_inner_knuckle.stl" />
         </geometry>
       </collision>
@@ -97,15 +103,16 @@
         <mass value="0.0104003125914103" />
         <inertia
-            ixx="2.71909453810972E-06"
-            ixy="1.35402465472579E-21"
-            ixz="-7.1817349065269E-22"
-            iyy="7.69100314106116E-07"
-            iyz="6.74715432769696E-07"
-            izz="2.30315190420171E-06" />
-      </inertial>
-      <visual>
-        <origin xyz="0 0 0" rpy="0 0 0" />
-        <geometry>
-          <mesh filename="file://$(find robotiq_description)/meshes/visual/2f_140/robotiq_2f_${stroke}_inner_finger.stl" />
+          ixx="2.71909453810972E-06"
+          ixy="1.35402465472579E-21"
+          ixz="-7.1817349065269E-22"
+          iyy="7.69100314106116E-07"
+          iyz="6.74715432769696E-07"
+          izz="2.30315190420171E-06" />
+      </inertial>
+      <visual>
+        <origin xyz="0 0 0" rpy="0 0 0" />
+        <geometry>
+          <mesh
+            filename="file://$(find robotiq_description)/meshes/visual/2f_140/robotiq_2f_${stroke}_inner_finger.stl" />
         </geometry>
         <material name="">
@@ -116,5 +123,6 @@
         <origin xyz="0 0 0" rpy="0 0 0" />
         <geometry>
-          <mesh filename="file://$(find robotiq_description)/meshes/collision/2f_140/robotiq_2f_${stroke}_inner_finger.stl" />
+          <mesh
+            filename="file://$(find robotiq_description)/meshes/collision/2f_140/robotiq_2f_${stroke}_inner_finger.stl" />
         </geometry>
       </collision>
@@ -127,5 +135,5 @@
         <origin xyz="0 0 0" rpy="0 0 0" />
         <geometry>
-          <box size="0.027 0.065 0.0075"/>
+          <box size="0.027 0.065 0.0075" />
         </geometry>
         <material name="">
@@ -136,5 +144,5 @@
         <origin xyz="0 0 0" rpy="0 0 0" />
         <geometry>
-           <box size="0.03 0.07 0.0075"/>
+          <box size="0.03 0.07 0.0075" />
         </geometry>
         <material name="">
@@ -151,6 +159,7 @@
       <axis xyz="-1 0 0" />
       <limit lower="0" upper="0.7" velocity="2.0" effort="1000" />
-    </joint>
-    <xacro:finger_joints prefix="${prefix}" fingerprefix="left" reflect="1.0"/>
+      <dynamics damping="2.0" friction="1.0" />
+    </joint>
+    <xacro:finger_joints prefix="${prefix}" fingerprefix="left" reflect="1.0" />
   </xacro:macro>
   <xacro:macro name="right_outer_knuckle_joint" params="prefix">
@@ -161,7 +170,8 @@
       <axis xyz="1 0 0" />
       <limit lower="-0.725" upper="0.725" velocity="2.0" effort="1000" />
-    <mimic joint="${prefix}finger_joint" multiplier="-1" offset="0" />
-    </joint>
-    <xacro:finger_joints prefix="${prefix}" fingerprefix="right" reflect="-1.0"/>
+      <mimic joint="${prefix}finger_joint" multiplier="-1" offset="0" />
+      <dynamics damping="2.0" friction="1.0" />
+    </joint>
+    <xacro:finger_joints prefix="${prefix}" fingerprefix="right" reflect="-1.0" />
   </xacro:macro>
   <xacro:macro name="outer_finger_joint" params="prefix fingerprefix">
@@ -175,5 +185,6 @@
   <xacro:macro name="inner_knuckle_joint" params="prefix fingerprefix reflect">
     <joint name="${prefix}${fingerprefix}_inner_knuckle_joint" type="revolute">
-      <origin xyz="0 ${reflect * -0.0127} 0.06142" rpy="${pi / 2 + .725} 0 ${(reflect - 1) * pi / 2}" />
+      <origin xyz="0 ${reflect * -0.0127} 0.06142"
+        rpy="${pi / 2 + .725} 0 ${(reflect - 1) * pi / 2}" />
       <parent link="${prefix}robotiq_140_base_link" />
       <child link="${prefix}${fingerprefix}_inner_knuckle" />
@@ -181,4 +192,5 @@
       <limit lower="-0.8757" upper="0.8757" velocity="2.0" effort="1000" />
       <mimic joint="${prefix}finger_joint" multiplier="-1" offset="0" />
+      <dynamics damping="2.0" friction="1.0" />
     </joint>
   </xacro:macro>
@@ -191,4 +203,5 @@
       <limit lower="-0.8757" upper="0.8757" velocity="2.0" effort="1000" />
       <mimic joint="${prefix}finger_joint" multiplier="1" offset="0" />
+      <dynamics damping="2.0" friction="1.0" />
     </joint>
   </xacro:macro>
@@ -202,15 +215,16 @@
   </xacro:macro>
   <xacro:macro name="finger_joints" params="prefix fingerprefix reflect">
-    <xacro:outer_finger_joint prefix="${prefix}" fingerprefix="${fingerprefix}"/>
-    <xacro:inner_knuckle_joint prefix="${prefix}" fingerprefix="${fingerprefix}" reflect="${reflect}"/>
-    <xacro:inner_finger_joint prefix="${prefix}" fingerprefix="${fingerprefix}"/>
-    <xacro:inner_finger_pad_joint prefix="${prefix}" fingerprefix="${fingerprefix}"/>
+    <xacro:outer_finger_joint prefix="${prefix}" fingerprefix="${fingerprefix}" />
+    <xacro:inner_knuckle_joint prefix="${prefix}" fingerprefix="${fingerprefix}"
+      reflect="${reflect}" />
+    <xacro:inner_finger_joint prefix="${prefix}" fingerprefix="${fingerprefix}" />
+    <xacro:inner_finger_pad_joint prefix="${prefix}" fingerprefix="${fingerprefix}" />
   </xacro:macro>
   <xacro:macro name="finger_links" params="prefix fingerprefix stroke">
-    <xacro:outer_knuckle prefix="${prefix}" fingerprefix="${fingerprefix}" stroke="${stroke}"/>
-    <xacro:outer_finger prefix="${prefix}" fingerprefix="${fingerprefix}" stroke="${stroke}"/>
-    <xacro:inner_finger prefix="${prefix}" fingerprefix="${fingerprefix}" stroke="${stroke}"/>
-    <xacro:inner_finger_pad prefix="${prefix}" fingerprefix="${fingerprefix}"/>
-    <xacro:inner_knuckle prefix="${prefix}" fingerprefix="${fingerprefix}" stroke="${stroke}"/>
+    <xacro:outer_knuckle prefix="${prefix}" fingerprefix="${fingerprefix}" stroke="${stroke}" />
+    <xacro:outer_finger prefix="${prefix}" fingerprefix="${fingerprefix}" stroke="${stroke}" />
+    <xacro:inner_finger prefix="${prefix}" fingerprefix="${fingerprefix}" stroke="${stroke}" />
+    <xacro:inner_finger_pad prefix="${prefix}" fingerprefix="${fingerprefix}" />
+    <xacro:inner_knuckle prefix="${prefix}" fingerprefix="${fingerprefix}" stroke="${stroke}" />
   </xacro:macro>
 </robot>

File: robotiq_description/urdf/robotiq_2f_140_macro.urdf.xacro (robot description, xacro)
@@ -56,6 +56,6 @@
           <!-- NOTE: This collision stl will cause collision in Gazebo -->
           <geometry>
-            <cylinder length="0.006" radius="0.2"/>
-            <!-- <mesh filename="file://$(find robotiq_description)/meshes/collision/2f_140/robotiq_2f_140_base_link.stl" /> -->
+            <!-- <cylinder length="0.006" radius="0.02"/> -->
+            <mesh filename="file://$(find robotiq_description)/meshes/collision/2f_140/robotiq_2f_140_base_link.stl" />
           </geometry>
         </collision>

Commit message: Added damping and friction property to ease value setting
Signed-off-by: laidvi <laidvi@schaeffler.com>

File: robotiq_description/urdf/robotiq_2f_140.xacro (robot description, xacro)
@@ -1,4 +1,6 @@
 <?xml version="1.0"?>
 <robot xmlns:xacro="http://ros.org/wiki/xacro">
+  <xacro:property name="damping" value="50.0" />
+  <xacro:property name="friction" value="1000.0" />
   <xacro:macro name="outer_knuckle" params="prefix fingerprefix stroke">
     <link name="${prefix}${fingerprefix}_outer_knuckle">
@@ -159,5 +161,5 @@
       <axis xyz="-1 0 0" />
       <limit lower="0" upper="0.7" velocity="2.0" effort="1000" />
-      <dynamics damping="2.0" friction="1.0" />
+      <dynamics damping="${damping}" friction="${friction}" />
     </joint>
     <xacro:finger_joints prefix="${prefix}" fingerprefix="left" reflect="1.0" />
@@ -171,5 +173,5 @@
       <limit lower="-0.725" upper="0.725" velocity="2.0" effort="1000" />
       <mimic joint="${prefix}finger_joint" multiplier="-1" offset="0" />
-      <dynamics damping="2.0" friction="1.0" />
+      <dynamics damping="${damping}" friction="${friction}" />
     </joint>
     <xacro:finger_joints prefix="${prefix}" fingerprefix="right" reflect="-1.0" />
@@ -192,5 +194,5 @@
       <limit lower="-0.8757" upper="0.8757" velocity="2.0" effort="1000" />
       <mimic joint="${prefix}finger_joint" multiplier="-1" offset="0" />
-      <dynamics damping="2.0" friction="1.0" />
+      <dynamics damping="${damping}" friction="${friction}" />
     </joint>
   </xacro:macro>
@@ -203,5 +205,5 @@
       <limit lower="-0.8757" upper="0.8757" velocity="2.0" effort="1000" />
       <mimic joint="${prefix}finger_joint" multiplier="1" offset="0" />
-      <dynamics damping="2.0" friction="1.0" />
+      <dynamics damping="${damping}" friction="${friction}" />
     </joint>
   </xacro:macro>
